Commit message: pacifica1.urdf: updated

File: src/cartographer_ros/cartographer_ros/urdf/pacifica1.urdf (robot description, URDF)
Before this commit: robot itri_van, 5 links, 4 joints
Joints:
- joint car_to_imu_mount: origin xyz=0 0 0 rpy=-0.07200409107649926 0.08272472913712309 0.018289895683322135 -> xyz=0 0 0 rpy=-0.014072329314525574 0.0365023826176044 -0.0339465024275643
